Commit message: Done Chasis body

File: description/robot_core.xacro (robot description, xacro)
@@ -15,3 +15,15 @@
     <link name="base_link">
     </link>
+    <joint name="chasis" type="fixed">
+        <parent link="base_link">
+        <child link="chasis">
+        <origin xyz="-0.1 0 0">
+    </joint>
+    <link name=:"chasis">
+        <origin xyz="0.15 0 0.075">
+        <visual>
+            <box size="0.3 0.3 0.15">
+            <material name ="blue">
+        </visual>
+    </link>
 </robot>

Commit message: Done Right Wheel

File: description/robot_core.xacro (robot description, xacro)
@@ -30,8 +30,8 @@
     </link>
     <!-- LEFT WHEEL LINK -->
-    <joint name="left_wheel_joint" type="continous">
+    <joint name="left_wheel_joint" type="continuous">
         <parent link="base_link"/>
-        <child  link="left_wheel"/>
-        <origin xyz=" 0 0.175 0" rpy="-${pi/2} 0 0" />
+        <child link="left_wheel"/>
+        <origin xyz="0 0.175 0" rpy="-1.5708 0 0" /> <!-- Assuming -pi/2 radians -->
         <axis xyz="0 0 1"/>
     </joint>
@@ -43,3 +43,19 @@
             <material name="white"/>
         </visual>
+    </link>
+    <!-- RIGHT WHEEL LINK -->
+    <joint name="right_wheel_joint" type="continuous">
+        <parent link="base_link"/>
+        <child link="right_wheel"/>
+        <origin xyz="0 -0.175 0" rpy="1.5708 0 0" /> <!-- Assuming pi/2 radians -->
+        <axis xyz="0 0 -1"/>
+    </joint>
+    <link name="right_wheel">
+        <visual>
+            <geometry>
+                <cylinder radius="0.05" length="0.04"/>
+            </geometry>
+            <material name="white"/>
+        </visual>
+    </link>
 </robot>

Commit message: Caster Wheel

File: description/robot_core.xacro (robot description, xacro)
@@ -15,10 +15,10 @@
     <link name="base_link">
     </link>
-    <joint name="chasis" type="fixed">
+    <joint name="chassis_joint" type="fixed">
         <parent link="base_link"/>
-        <child link="chasis"/>
+        <child link="chassis"/>
         <origin xyz="-0.1 0 0"/>
     </joint>
-    <link name="chasis">
+    <link name="chassis">
         <visual>
             <origin xyz="0.15 0 0.075"/>
@@ -59,3 +59,17 @@
         </visual>
     </link>
+    <!-- CASTER WHEEL LINK -->
+    <joint name="caster_wheel_joint" type="fixed">
+        <parent link="chassis"/>
+        <child link="caster_wheel"/>
+        <origin xyz="0.24 0 0" />
+    </joint>
+     <link name="caster_wheel">
+        <visual>
+            <geometry>
+                <sphere radius="0.05" />
+            </geometry>
+            <material name="black"/>
+        </visual>
+    </link>
 </robot>

Commit message: Added Collision

File: description/robot_core.xacro (robot description, xacro)
@@ -28,4 +28,10 @@
             <material name="blue"/>
         </visual>
+        <collision>
+            <origin xyz="0.15 0 0.075"/>
+            <geometry>
+                <box size="0.3 0.3 0.15"/>
+            </geometry>
+        </collision>
     </link>
     <!-- LEFT WHEEL LINK -->
@@ -43,4 +49,9 @@
             <material name="white"/>
         </visual>
+        <collision>
+            <geometry>
+                <cylinder radius="0.05" length="0.04"/>
+            </geometry>
+        </collision>
     </link>
     <!-- RIGHT WHEEL LINK -->
@@ -58,4 +69,9 @@
             <material name="white"/>
         </visual>
+        <collision>
+            <geometry>
+                <cylinder radius="0.05" length="0.04"/>
+            </geometry>
+        </collision>
     </link>
     <!-- CASTER WHEEL LINK -->
@@ -72,4 +88,9 @@
             <material name="black"/>
         </visual>
+        <collision>
+            <geometry>
+                <sphere radius="0.05"/>
+            </geometry>
+        </collision>
     </link>
 </robot>

Commit message: Done intertias

File: description/robot_core.xacro (robot description, xacro)
@@ -1,4 +1,5 @@
 <?xml version="1.0"?>
 <robot xmlns:xacro="http://www.ros.org/wiki/xacro">
+    <xacro:include filename="inertial_macro.xacro" />
     <material name="white">
         <color rgba="1 1 1 1"/>
@@ -34,4 +35,7 @@
             </geometry>
         </collision>
+        <xacro:inertial_box mass="0.5" x="0.3" y="0.3" z="0.15">
+            <origin xyz="0.15 0 0.075" rpy="0 0 0"/>
+        </xacro:inertial_box>
     </link>
     <!-- LEFT WHEEL LINK -->
@@ -54,4 +58,7 @@
             </geometry>
         </collision>
+        <xacro:inertial_cylinder mass="0.1" radius="0.05" length="0.04">
+            <origin xyz="0 0 0" rpy="0 0 0"/>
+        </xacro:inertial_cylinder>
     </link>
     <!-- RIGHT WHEEL LINK -->
@@ -74,4 +81,7 @@
             </geometry>
         </collision>
+        <xacro:inertial_cylinder mass="0.1" radius="0.05" length="0.04">
+            <origin xyz="0 0 0" rpy="0 0 0"/>
+        </xacro:inertial_cylinder>
     </link>
     <!-- CASTER WHEEL LINK -->
@@ -93,4 +103,7 @@
             </geometry>
         </collision>
+        <xacro:inertial_sphere mass="0.1" radius="0.05">
+            <origin xyz="0 0 0" rpy="0 0 0"/>
+        </xacro:inertial_sphere>
     </link>
 </robot>

Commit message: Added launch file

File: description/robot_core.xacro (robot description, xacro)
@@ -39,4 +39,7 @@
         </xacro:inertial_box>
     </link>
+    <gazebo reference="chassis">
+        <material>Gazebo/white</material>
+    </gazebo>
     <!-- LEFT WHEEL LINK -->
     <joint name="left_wheel_joint" type="continuous">

Commit message: Added Gazerbo stuff

File: description/robot_core.xacro (robot description, xacro)
@@ -40,5 +40,5 @@
     </link>
     <gazebo reference="chassis">
-        <material>Gazebo/white</material>
+        <material>Gazebo/Blue</material>
     </gazebo>
     <!-- LEFT WHEEL LINK -->
@@ -65,4 +65,7 @@
         </xacro:inertial_cylinder>
     </link>
+    <gazebo reference="left_wheel">
+        <material>Gazebo/White</material>
+    </gazebo>
     <!-- RIGHT WHEEL LINK -->
     <joint name="right_wheel_joint" type="continuous">
@@ -88,4 +91,7 @@
         </xacro:inertial_cylinder>
     </link>
+    <gazebo reference="right_wheel">
+        <material>Gazebo/White</material>
+    </gazebo>
     <!-- CASTER WHEEL LINK -->
     <joint name="caster_wheel_joint" type="fixed">
@@ -110,3 +116,6 @@
         </xacro:inertial_sphere>
     </link>
+    <gazebo reference="caster_wheel">
+        <material>Gazebo/Black</material>
+    </gazebo>
 </robot>
